File: pcb/lipo-charger/lipo-charger.kicad_sch (KiCad schematic)
At the start: 12 parts, among them J1 USB_B_Micro, J2 BATTERY, J3 OUTPUT, SW1 BATTERY_EN, U1 MCP73831-2-OT

Commit message: update BOMs for JLC assembly
Parts:
- C1, C2: JLC (none) -> 0805; JLCSC (none) -> C1779; JLCSC Part # (none) -> C1779; Part Number (none) -> CC0805KKX7R6BB475
- D1: JLC (none) -> 1206; JLCSC (none) -> C434438; JLCSC Part # (none) -> C434438
- D2: JLC (none) -> SOD-323; JLCSC (none) -> C490614; JLCSC Part # (none) -> C490614; Part Number SD05C-7 -> Leiditech SD05
- D3: JLC (none) -> SOD-123FL; JLCSC (none) -> C669022; JLCSC Part # (none) -> C669022; Part Number NRVB120VLSF -> SM5817PL-TP
- J2, J3: JLCSC Part # (none) -> C5251182
- R1: JLC (none) -> 0805; JLCSC (none) -> C17655; JLCSC Part # (none) -> C17655; Part Number (none) -> RC0805FR-07390RL
- R2: JLC (none) -> 0805; JLCSC (none) -> C4328; Part Number (none) -> RC0805FR-0720KL
- SW1: JLCSC Part # (none) -> C273395
- U1: JLC (none) -> SOT-23-5; JLCSC (none) -> C424093; JLCSC Part # (none) -> C424093
